File: MAIN/MAIN.kicad_pcb (KiCad board)
At the start: 6 copper layers, 174.6 x 124.6 mm, 388 parts, among them IC2 SN74LV1T126DCKRG4, J1 B14B-PASK-1__LF__SN_, J10 B07B-PASK-1, J11 B03B-PASK-1_LF__SN_, J12 B14B-PASK-1__LF__SN_, J13 B14B-PASK-1__LF__SN_, J14 B14B-PASK-1__LF__SN_, J2 2601-3102, J3 2601-3102, J4 B05B-PASK-1, J5 B05B-PASK-1, J6 FTSH-105-X-X-DV-007-P-X, J7 USB4085-GF-A_REVB, J8 MSD-4-A, J9 B07B-PASK-1, K1 AGQ200A06, K2 AGQ200A06, K3 AGQ200A06, K4 AGQ200A06, K5 AGQ200A06, K6 AGQ200A06, K7 AGQ200A06, K8 AGQ200A06, Q1 SI7252DP-T1-GE3, Q2 2N7002K, Q3 2N7002K, Q4 2N7002K, Q5 2N7002K, Q6 2N7002K, Q7 2N7002K, Q8 2N7002K, Q9 2N7002K, U1 LTC4367HDD-TRPBF, U10 MCP9601T-E/MX, U11 SN74LVC1G32DSF2, U12 MCP9601T-E/MX, U13 SN74LVC1G32DSF2, U14 MCP9601T-E/MX, U15 SN74LVC1G32DSF2, U16 MCP9601T-E/MX, U17 SN74LVC1G32DSF2, U18 MCP9601T-E/MX, U19 SN74LVC1G32DSF2, U2 REF3133AIDBZR, U20 MCP9601T-E/MX, U21 SN74LVC1G32DSF2, U22 MCP9601T-E/MX, U23 SN74LVC1G32DSF2, U24 USBLC6-2SC6, U25 GD25Q64ETIGR, U3 MAX17634BATP+, U4 AP63203WU-7, U5 AP63201WU-7, U6 NAU7802SGI, U7 NAU7802SGI, U8 MCP9601T-E/MX, U9 SN74LVC1G32DSF2, Y1 32.7680kHz

Commit message: stuff
Routing:
- net (no net): track 0.00 -> 69.4 mm
Changed lines of the file:
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@@
+	)
+	(segment
+		(start 256.18 51.45)
+		(end 256.18 55.94)
+		(width 0.1)
+		(layer "F.Cu")
+		(net 0)
+	)
+	(segment
+		(start 258.73 57.57)
+		(end 258.73 75.11)
+		(width 0.1)
+		(layer "F.Cu")
+		(net 0)
+	)
+	(segment
+		(start 264.23 74.09)
+		(end 264.23 57.26)
+		(width 0.1)
+		(layer "F.Cu")
+		(net 0)
+	)
+	(segment
+		(start 258.73 75.11)
+		(end 260.97 77.35)
+		(width 0.1)
+		(layer "F.Cu")
+		(net 0)
+	)
+	(segment
+		(start 258.42 51.45)
+		(end 256.18 51.45)
+		(width 0.1)
+		(layer "F.Cu")
+		(net 0)
+	)
+	(segment
+		(start 256.18 55.94)
+		(end 254.65 57.47)
+		(width 0.1)
+		(layer "F.Cu")
+		(net 0)
+	)
+	(segment
+		(start 260.97 77.35)
+		(end 264.23 74.09)
+		(width 0.1)
+		(layer "F.Cu")
+		(net 0)
+	)
+	(segment
+		(start 264.23 57.26)
+		(end 258.42 51.45)
+		(width 0.1)
+		(layer "F.Cu")
+		(net 0)
+	)
+	(segment
+		(start 254.65 57.47)
+		(end 254.65 67.66)
+		(width 0.1)
+		(layer "F.Cu")
+		(net 0)
 	)
 	(segment
