File: MAIN/page3.kicad_sch (KiCad schematic)
At the start: 11 parts, among them J4 B05B-PASK-1, U26 INA333xxDRG, U6 NAU7802SGI

Commit message: changed
changed
Parts:
- added C1: C_Small, symbol Device:C_Small
Changed lines of the file:
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@@
 			"RgAvAHIAZgBIADgAbgBlAGYAOABWAGkAOQA2AEkAYQBCAEkASQBtAEkARQB0AEMAMABYAFQAZQA3"
 			"AGkATQBnAHkANgAvAGQAZAA5ADkAOQBkAGkAdABaAFIANwBzAFgAOQAyAFoAdgBPAGwAOQByAGUA"
-			"eAB1AGUAVQBIAGYAVwBNAFMAZwBPAGcAUgB3AEoANgBPAGoAZABWADAAKw=="
+			"eAB1AGUAVQBIAGYAVwBNAFMAZwBPAGcAUgB3AEoANgBPAGoAZABWADAAKwBOAHMAbABOAFMAUQA4"
+			"ADEARwBFAEwAQwBLAFEARgBxAGwALwBpAGoAdgBaAFoAWABiAFUAUQBZAEMARQBMAGkATQBRAEkA"
+			"aQBsAHYAbgBUAFQAZQBmADAAWgBrAE8AdgBQAHAAVQBQAGkAUgBUAEIARgBBADEAYwBCAEYAWgBy"
+			"AFIAdQAzAFQAeQAwAEIAVQBDAEUARQBpAE4AZwBNADcATwAwAEYAawBhAEkAWQA3AEwAcwAxAFAA"
+			"VwBUADYAKwAxAEMAbwBQAHAAZwBNAGYAVAAvAFIAMQBXADIAWQBzAHkARQBJAEIAQQBQAEEASQA2"
+			"AGkASwBJAGYAMABPAHQAKwBIAEwAcgBSAE8AYwBOAGUAQQBxAE4ARwBqAFoATAAxADYAOQBjAFgA"
+			"cABXAEMAVwBwAGIANABxADEAYQAvAEMAegBUAGUATQBLAFUAcgBmAE8ASgBQAEoAVABvAGwARABq"
+			"ADcAVQBRAFMASgBiAEEAUQAyAHUAYQBrAHgAVgBZAFEASgByAHAAYwBsACsAVQA5ADAAcgBWAG4A"
+			"VwB3AEcAQQBRAGkAVQBRAE8AQgAzAGYAKwAvADEARQBsAGEANQB1ADIAUQBvAEsAMABVADkAdQA5"
+			"AGYAUAA3ADAAZgA4AGMAOABrADYAYgA0AEkAcABGADYARgA3AFUAWAB2AE4AcABRAE8ARQByAGgA"
+			"QwBBAGcAUAAwAEUAbgBuADAAaABqAEsAYgB6AHUAVAB3AHgAUABEAHYAbAB3AFoAUgAvAEwATwBZ"
+			"ADcASABXAGsARQBPAHYAbwBYAFIAQwA4AHgAWQAvADkASgBSAGsATQBJAFEARQBBAC8AYgBCADgA"
+			"MwBiAHAAegBvAEIAdQBjAE0AdQB3AG4AbwBZAEoAZgBPAFQAaABrADkAZQBuAFIAawBSAGIATQBz"
+			"ADkAWABYAEcAWQBLAFoAawBMAGcAQwBtAEgANgBoAEcAQgBzADkARQBDAEEAUgBPAG8ASwAvAGoA"
+			"dwA3AEsANABhAGEAQQB3AFgAZQA2AEwAOABsADUAcABlAEoARQA5AEkAQQBDAEIATwBBAFMAcQBU"
+			"AHAAeQA1AHAAQwBSADUASABGAGsAdQByAE4AVgBaAEsAUwA3AG8ARwBWAFYASAByADQASQBwAGwA"
+			"UAB1AEsANgBuAGIAbQBRAFEAQQBDAG8AUgBEAFEAVwBTAGsAMQBKADgATgBwAE8AagArAFMAWAA0"
+			"AGQAbgBwADYAeQBkAGEAawA5AG0AUwBoAHEAQgBEAHQAMgBJAG4AZwBFAEIAQwBQAGgAQgBvAEwA"
+			"YQAyAFYAbABhAHUAWABDAGsAMQBOAGUAbQBWAFkAdgBLAEQAWABEAFoAVw=="
 		)
 	)
@@
 					(unit 1)
 				)
+			)
+		)
+	)
+	(symbol
+		(lib_id "Device:C_Small")
+		(at 125.73 49.53 0)
+		(unit 1)
+		(exclude_from_sim no)
+		(in_bom yes)
+		(on_board yes)
+		(dnp no)
+		(fields_autoplaced yes)
+		(property "Reference" "C1"
+			(at 128.27 48.2662 0)
+			(effects
+				(font
+					(size 1.27 1.27)
+				)
+				(justify left)
+			)
+		)
+		(property "Value" "C_Small"
+			(at 128.27 50.8062 0)
+			(effects
+				(font
+					(size 1.27 1.27)
+				)
+				(justify left)
+			)
+		)
+		(property "Footprint" ""
+			(at 125.73 49.53 0)
+			(effects
+				(font
+					(size 1.27 1.27)
+				)
+				(hide yes)
+			)
+		)
+		(property "Datasheet" "~"
+			(at 125.73 49.53 0)
+			(effects
+				(font
+					(size 1.27 1.27)
+				)
+				(hide yes)
+			)
+		)
+		(property "Description" "Unpolarized capacitor, small symbol"
+			(at 125.73 49.53 0)
+			(effects
+				(font
+					(size 1.27 1.27)
+				)
+				(hide yes)
+			)
+		)
+		(pin "1"
+		)
+		(pin "2"
+		)
+		(instances
+			(project ""
+				(path "/906e79d2-f21c-41e4-84cb-e799c410b05f/74454ce8-b9af-4706-9252-bd7bd1e06e51"
+					(reference "C1")
+					(unit 1)
+				)
+				(path "/906e79d2-f21c-41e4-84cb-e799c410b05f/87e1a79d-c764-4fd6-83c5-39297e9d65b4"
+					(reference "C3")
+					(unit 1)
+				)

Commit message: update cap
Parts:
- added C88, C90: C_Small, symbol Device:C_Small
Changed lines of the file:
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@@
+	)
+	(symbol
+		(lib_id "Device:C_Small")
+		(at 106.68 74.93 0)
+		(unit 1)
+		(exclude_from_sim no)
+		(in_bom yes)
+		(on_board yes)
+		(dnp no)
+		(fields_autoplaced yes)
+		(property "Reference" "C90"
+			(at 109.22 73.6662 0)
+			(effects
+				(font
+					(size 1.27 1.27)
+				)
+				(justify left)
+			)
+		)
+		(property "Value" "C_Small"
+			(at 109.22 76.2062 0)
+			(effects
+				(font
+					(size 1.27 1.27)
+				)
+				(justify left)
+			)
+		)
+		(property "Footprint" ""
+			(at 106.68 74.93 0)
+			(effects
+				(font
+					(size 1.27 1.27)
+				)
+				(hide yes)
+			)
+		)
+		(property "Datasheet" "~"
+			(at 106.68 74.93 0)
+			(effects
+				(font
+					(size 1.27 1.27)
+				)
+				(hide yes)
+			)
+		)
+		(property "Description" "Unpolarized capacitor, small symbol"
+			(at 106.68 74.93 0)
+			(effects
+				(font
+					(size 1.27 1.27)
+				)
+				(hide yes)
+			)
+		)
+		(pin "1"
+		)
+		(pin "2"
+		)
+		(instances
+			(project "MAIN"
+				(path "/906e79d2-f21c-41e4-84cb-e799c410b05f/74454ce8-b9af-4706-9252-bd7bd1e06e51"
+					(reference "C90")
+					(unit 1)
+				)
+				(path "/906e79d2-f21c-41e4-84cb-e799c410b05f/87e1a79d-c764-4fd6-83c5-39297e9d65b4"
+					(reference "C91")
+					(unit 1)
+				)
+			)
+		)
 	)
 	(symbol
@@
 					(unit 1)
 				)
+			)
+		)
+	)
+	(symbol
+		(lib_id "Device:C_Small")
+		(at 81.28 92.71 0)
+		(unit 1)
+		(exclude_from_sim no)
+		(in_bom yes)
+		(on_board yes)
+		(dnp no)
+		(fields_autoplaced yes)
+		(property "Reference" "C88"
+			(at 83.82 91.4462 0)
+			(effects
+				(font
+					(size 1.27 1.27)
+				)
+				(justify left)
+			)
+		)
+		(property "Value" "C_Small"
+			(at 83.82 93.9862 0)
+			(effects
+				(font
+					(size 1.27 1.27)
+				)
+				(justify left)
+			)
+		)
+		(property "Footprint" ""
+			(at 81.28 92.71 0)
+			(effects
+				(font
+					(size 1.27 1.27)
+				)
+				(hide yes)
+			)
+		)
+		(property "Datasheet" "~"
+			(at 81.28 92.71 0)
+			(effects
+				(font
+					(size 1.27 1.27)
+				)
+				(hide yes)
+			)
+		)
+		(property "Description" "Unpolarized capacitor, small symbol"
+			(at 81.28 92.71 0)
+			(effects
+				(font
+					(size 1.27 1.27)
+				)
+				(hide yes)
+			)
+		)
+		(pin "1"
+		)
+		(pin "2"
+		)
+		(instances
+			(project "MAIN"
+				(path "/906e79d2-f21c-41e4-84cb-e799c410b05f/74454ce8-b9af-4706-9252-bd7bd1e06e51"
+					(reference "C88")
+					(unit 1)
+				)
+				(path "/906e79d2-f21c-41e4-84cb-e799c410b05f/87e1a79d-c764-4fd6-83c5-39297e9d65b4"
+					(reference "C89")
+					(unit 1)
+				)

Commit message: sdfghjkl;
Parts:
- removed C1, C88, C90: C_Small, symbol Device:C_Small
Connections:
- net GND: now also U26.4 (V-), U26.5 (Ref), U26.9 (EP)
